Commit message: Model changes and rebuilding the drive nodes from the ground up
A number of problems were found with the drivenode.py implementation.  I decided to start
from the beginning writing a drive node based on arbotix.  I was able to get a simulated
node to move the model in rviz.  From there, I was able to add basic message handling from
the halnode and to see the real arlobot visualized in rviz.  Additionally, there were
problems found in the Psoc code where the angular velocity was being used without first
being convered to meters/second.  This showed up when attempt to do isolated moves, e.g.,
moving in a straight line.  In which case the linear velocity of the wheels was not the
same as the linear velocity of the unicycle model -- an impossibility if we're to get
accurate motion.  Anyway, the psoc code is fixed and now I need to build up the drive
node and the rest of the arlobot model.

File: arlobot_description/urdf/arlobot.base.urdf.xacro (robot description, xacro)
@@ -39,12 +39,15 @@
     </macro>
     <macro name="wheel" params="parent suffix reflect color">
-        <!-- Note: type is fixed here.  tried continuous but then the link is lost.  not sure why though -->
+        <!-- Note: type is fixed.  continuous is possible but then joint_states would need to be published.  For
+        visualization its not particularly necessary to have the wheels turn.  Maybe in Gazebo simulation it will be
+        required.  If that is the case, then of course something in Arlobot mobile base will need to publish the
+        joint_states.
+         -->
         <joint name="${parent}_${suffix}_wheel_joint" type="fixed">
-            <axis xyz="0 0 1" />
-            <limit effort="100" velocity="100"/>
-            <safety_controller k_velocity="10" />
-            <origin xyz="${wheel_offset_x} ${reflect*wheel_offset_y} ${wheel_offset_z}" rpy="${reflect*PI/2} 0 0" />
             <parent link="${parent}_link"/>
             <child link="${suffix}_wheel_link"/>
+            <origin xyz="${wheel_offset_x} ${reflect*wheel_offset_y} ${wheel_offset_z}" rpy="${reflect*PI/2} 0 0" />
+            <limit effort="0.1" velocity="0.01"/>
+            <axis xyz="0 0 1" />
         </joint>
         <link name="${suffix}_wheel_link">

File: arlobot_description/urdf/arlobot.test.urdf.xacro (robot description, xacro)
@@ -5,11 +5,5 @@
     <xacro:include filename="$(find arlobot_description)/urdf/arlobot.global.urdf.xacro"/>
     <xacro:include filename="$(find arlobot_description)/urdf/arlobot.base.urdf.xacro" />
-    <xacro:include filename="$(find arlobot_description)/urdf/arlobot.baselevel.urdf.xacro" />
-    <xacro:include filename="$(find arlobot_description)/urdf/arlobot.midlevel.urdf.xacro" />
-    <xacro:include filename="$(find arlobot_description)/urdf/arlobot.toplevel.urdf.xacro" />
     <!-- Add each level of the robot -->
     <base color="Black"/>
-    <baselevel parent="base" name="baselevel" color="Black"/>
-    <midlevel parent="baselevel" name="midlevel" color="Black"/>
-    <toplevel parent="midlevel" name="toplevel" color="Black"/>
 </robot>
